Commit message: feat(ROS1): made changes in order to run with ROS1 noetic

File: urdf/ur5_rg2.urdf (robot description, URDF)
Before this commit: robot ur5_rg2, 11 links, 10 joints
Links:
- added link world, mass 0.0
- link base_link: mass None -> 4.210389694173812; geometry collision mesh filename=package://ur5_rg2_ign/ur5_rg2/meshes/collision/ur5/base.stl; visual mesh filename=package://ur5_rg2_ign/ur5_rg2/meshes/visual/ur5/base.dae
- link forearm_link: mass None -> 2.275; geometry collision mesh filename=package://ur5_rg2_ign/ur5_rg2/meshes/collision/ur5/forearm.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; visual mesh filename=package://ur5_rg2_ign/ur5_rg2/meshes/visual/ur5/forearm.dae
- link rg2_hand: mass None -> 0.5; geometry collision mesh filename=package://ur5_rg2_ign/ur5_rg2/meshes/collision/rg2/hand.stl; visual mesh filename=package://ur5_rg2_ign/ur5_rg2/meshes/visual/rg2/hand.dae
- link rg2_leftfinger: mass None -> 0.1; geometry collision mesh filename=package://ur5_rg2_ign/ur5_rg2/meshes/collision/rg2/finger.s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; visual mesh filename=package://ur5_rg2_ign/ur5_rg2/meshes/visual/rg2/finger.dae
- link rg2_rightfinger: mass None -> 0.1; geometry collision mesh filename=package://ur5_rg2_ign/ur5_rg2/meshes/collision/rg2/finger.s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; visual mesh filename=package://ur5_rg2_ign/ur5_rg2/meshes/visual/rg2/finger.dae
- link shoulder_link: mass None -> 2.6078628081050645; geometry collision mesh filename=package://ur5_rg2_ign/ur5_rg2/meshes/collision/ur5/shoulder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; visual mesh filename=package://ur5_rg2_ign/ur5_rg2/meshes/visual/ur5/shoulder.dae
- link tool0: mass None -> 0.001
- link upper_arm_link: mass None -> 9.034556202946057; geometry collision mesh filename=package://ur5_rg2_ign/ur5_rg2/meshes/collision/ur5/upperarm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; visual mesh filename=package://ur5_rg2_ign/ur5_rg2/meshes/visual/ur5/upperarm.dae
- link wrist_1_link: mass None -> 0.8652783044597422; geometry collision mesh filename=package://ur5_rg2_ign/ur5_rg2/meshes/collision/ur5/wrist1.s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; visual mesh filename=package://ur5_rg2_ign/ur5_rg2/meshes/visual/ur5/wrist1.dae
- link wrist_2_link: mass None -> 1.219; geometry collision mesh filename=package://ur5_rg2_ign/ur5_rg2/meshes/collision/ur5/wrist2.s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; visual mesh filename=package://ur5_rg2_ign/ur5_rg2/meshes/visual/ur5/wrist2.dae
- link wrist_3_link: mass None -> 0.1879; geometry collision mesh filename=package://ur5_rg2_ign/ur5_rg2/meshes/collision/ur5/wrist3.s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; visual mesh filename=package://ur5_rg2_ign/ur5_rg2/meshes/visual/ur5/wrist3.dae
Joints:
- added joint world_joint: type fixed, parent world, child base_link, origin xyz=0 0 0 rpy=0 0 0
- joint rg2_finger_joint2: mimic joint=panda_finger_joint1 -> joint=rg2_finger_joint1 multiplier=1.0 offset=0.0
